Commit message: Updated inertia and damping matrix

File: vrx_urdf/wamv_description/urdf/wamv_base.urdf.xacro (robot description, xacro)
@@ -104,6 +104,6 @@
     <inertial>
       <!-- From WAM-V spec sheet -->
-      <mass value="180.0"/>
-      <inertia ixx="120.0" ixy="0.0" ixz="0.0" iyy="393" iyz="0.0" izz="446.0"/>
+      <mass value="70.0"/>
+      <inertia ixx="90.5" ixy="0.0" ixz="0.0" iyy="167.5" iyz="12.25" izz="42.65"/>
     </inertial>
   </link>

File: vrx_urdf/wamv_gazebo/urdf/dynamics/wamv_gazebo_dynamics_plugin.xacro (robot description, xacro)
@@ -45,15 +45,15 @@
         <nDotR>0.0</nDotR>
         <!-- Linear and quadratic drag -->
-        <xU>100.0</xU>
-        <xUU>150.0</xUU>
-        <yV>100.0</yV>
-        <yVV>100.0</yVV>
-        <zW>500.0</zW>
-        <kP>300.0</kP>
-        <kPP>600.0</kPP>
-        <mQ>900.0</mQ>
-        <mQQ>900.0</mQQ>
-        <nR>800.0</nR>
-        <nRR>800.0</nRR>
+        <xU>77.55</xU>
+        <xUU>75.0</xUU>
+        <yV>162.5</yV>
+        <yVV>75.0</yVV>
+        <zW>42.65</zW>
+        <kP>200.0</kP>
+        <kPP>300.0</kPP>
+        <mQ>450.0</mQ>
+        <mQQ>450.0</mQQ>
+        <nR>400.0</nR>
+        <nRR>400.0</nRR>
       </plugin>
     </gazebo>
