Commit message: Added Njord tasks

File: vrx_urdf/wamv_description/urdf/cpu_cases.xacro (robot description, xacro)
@@ -3,5 +3,5 @@
 <xacro:macro name="cpu_cases" params="position:='0 0 0' orientation:='0 0 0'">
   <link name="${namespace}/cpu_cases_link">
-    <visual>
+    <!-- <visual>
       <origin xyz="0.073 0 -1.53" rpy="0 0 0"/>
       <geometry>
@@ -20,5 +20,5 @@
         <box size="0.375 0.64 0.28"/>
       </geometry>
-    </collision>
+    </collision> -->
     <inertial>
       <mass value="20"/>
@@ -38,5 +38,5 @@
   </joint>
   <gazebo reference="${namespace}/cpu_cases_link">
-    <visual>
+    <!-- <visual>
       <material>
         <diffuse>1.0 1.0 1.0</diffuse>
@@ -51,5 +51,5 @@
         </pbr>
       </material>
-    </visual>
+    </visual> -->
   </gazebo>
 </xacro:macro>
